File: hw/with-vreg.sch (EAGLE design)
At the start: 10 parts

Commit message: hw: fixed 1k5 pull-up to be controlled by D5
Some lines of errors happened when the 1k5 pull-up from `D-`
wired directly to 3V3.

Think it caused by boot delay of Arduino.
Anyway, the errors can be removed by wire the pull-up to D5 and,
let UsbKeyboard control it.

Signed-off-by: Homin Lee <homin.lee@suapapa.net>
Parts:
- removed JP1: (no value), pinhead:PINHD-1X4
- removed X1: (no value), con-berg:PN61729
- added JP3: (no value), pinhead:PINHD-1X5
- added X2: (no value), con-berg:PN61729
Connections:
- new net N$4: JP3.1, R3.1
- net D+: now also JP2.3, X2.3; no longer JP2.2, X1.3
- net D-: now also JP2.2, R3.2, X2.2; no longer JP2.3, R3.1, X1.2
- net GND: now also JP3.5, X2.4; no longer JP1.4, X1.4
- net N$1: now also JP3.3; no longer JP1.2
- net N$2: now also JP3.4; no longer JP1.3
- net N$3: now also X2.1; no longer X1.1
- net VCC: now also JP3.2; no longer JP1.1, R3.2
Other:
- moved on the sheet: JP2, R3
